File: cycle_computer/cycle_computer.sch (KiCad schematic (older format))
At the start: 9 parts, among them Q1 Q_PMOS_DGS, Q2 Q_PMOS_DGS, Q3 Q_PMOS_DGS, Q4 Q_PMOS_DGS, U1 Wemos_LoLin32, U2 AdafruitUltimateGps, U3 MPL3115A2_breakout, U4 MPU9250_breakout, U5 st7745r_breakout

Commit message: Change to N-FETs
Parts:
- removed Q1, Q2, Q3, Q4: Q_PMOS_DGS, symbol q_pmos_dgs:Q_PMOS_DGS
- added Q1, Q2, Q3, Q4: Q_NMOS_DGS, symbol q_nmos_dgs:Q_NMOS_DGS
Changed lines of the file:
@@
 EESchema Schematic File Version 4
+LIBS:cycle_computer-cache
 EELAYER 26 0
 EELAYER END
@@
 Wire Wire Line
 	4700 3200 5200 3200
-$Comp
-L q_pmos_dgs:Q_PMOS_DGS Q2
-U 1 1 5BC2C1D7
+Wire Wire Line
+	4500 4000 4500 4600
+Wire Wire Line
+	4500 4600 4550 4600
+Wire Wire Line
+	4550 4600 4550 5550
+Connection ~ 4550 5550
+Wire Wire Line
+	4550 5550 4650 5550
+Wire Wire Line
+	4800 4200 5350 4200
+Wire Wire Line
+	5350 4200 5350 4150
+Wire Wire Line
+	5350 4150 5550 4150
+Wire Wire Line
+	4800 4200 4800 5450
+Wire Wire Line
+	4800 5450 5550 5450
+Wire Wire Line
+	4800 3800 4800 3750
+Wire Wire Line
+	4800 3750 4350 3750
+Wire Wire Line
+	4350 3750 4350 4400
+Connection ~ 4350 4400
+$Comp
+L q_nmos_dgs:Q_NMOS_DGS Q2
+U 1 1 5BC739F8
 P 4050 2450
-F 0 "Q2" H 4256 2496 50  0000 L CNN
-F 1 "Q_PMOS_DGS" H 4256 2405 50  0000 L CNN
+F 0 "Q2" H 4255 2404 50  0000 L CNN
+F 1 "Q_NMOS_DGS" H 4255 2495 50  0000 L CNN
 F 2 "" H 4250 2550 50  0001 C CNN
 F 3 "~" H 4050 2450 50  0001 C CNN
 	1    4050 2450
-	1    0    0    -1
-$EndComp
-$Comp
-L q_pmos_dgs:Q_PMOS_DGS Q3
-U 1 1 5BC2C39A
+	1    0    0    1
+$EndComp
+$Comp
+L q_nmos_dgs:Q_NMOS_DGS Q4
+U 1 1 5BC7DA03
 P 6100 2550
-F 0 "Q3" H 6306 2504 50  0000 L CNN
-F 1 "Q_PMOS_DGS" H 6306 2595 50  0000 L CNN
+F 0 "Q4" H 6306 2596 50  0000 L CNN
+F 1 "Q_NMOS_DGS" H 6306 2505 50  0000 L CNN
 F 2 "" H 6300 2650 50  0001 C CNN
 F 3 "~" H 6100 2550 50  0001 C CNN
 	1    6100 2550
-	-1   0    0    1
-$EndComp
-$Comp
-L q_pmos_dgs:Q_PMOS_DGS Q1
-U 1 1 5BC2C576
+	-1   0    0    -1
+$EndComp
+$Comp
+L q_nmos_dgs:Q_NMOS_DGS Q3
+U 1 1 5BC807E1
+P 4700 4000
+F 0 "Q3" H 4905 4046 50  0000 L CNN
+F 1 "Q_NMOS_DGS" H 4905 3955 50  0000 L CNN
+F 2 "" H 4900 4100 50  0001 C CNN
+F 3 "~" H 4700 4000 50  0001 C CNN
+	1    4700 4000
+	1    0    0    -1
+$EndComp
+Connection ~ 4800 4200
+$Comp
+L q_nmos_dgs:Q_NMOS_DGS Q1
+U 1 1 5BC8095B
 P 3400 5950
-F 0 "Q1" H 3606 5904 50  0000 L CNN
-F 1 "Q_PMOS_DGS" H 3606 5995 50  0000 L CNN
+F 0 "Q1" H 3605 5996 50  0000 L CNN
+F 1 "Q_NMOS_DGS" H 3605 5905 50  0000 L CNN
 F 2 "" H 3600 6050 50  0001 C CNN
 F 3 "~" H 3400 5950 50  0001 C CNN
 	1    3400 5950
-	1    0    0    1
-$EndComp
-$Comp
-L q_pmos_dgs:Q_PMOS_DGS Q4
-U 1 1 5BC2C79D
-P 4700 4000
-F 0 "Q4" H 4906 3954 50  0000 L CNN
-F 1 "Q_PMOS_DGS" H 4906 4045 50  0000 L CNN
-F 2 "" H 4900 4100 50  0001 C CNN
-F 3 "~" H 4700 4000 50  0001 C CNN
-	1    4700 4000
-	1    0    0    1
-$EndComp
-Wire Wire Line
-	4500 4000 4500 4600
-Wire Wire Line
-	4500 4600 4550 4600
-Wire Wire Line
-	4550 4600 4550 5550
-Connection ~ 4550 5550
-Wire Wire Line
-	4550 5550 4650 5550
-Wire Wire Line
-	4800 4200 5350 4200
-Wire Wire Line
-	5350 4200 5350 4150
-Wire Wire Line
-	5350 4150 5550 4150
-Wire Wire Line
-	4800 4200 4800 5450
-Wire Wire Line
-	4800 5450 5550 5450
-Connection ~ 4800 4200
-Wire Wire Line
-	4800 3800 4800 3750
-Wire Wire Line
-	4800 3750 4350 3750
-Wire Wire Line
-	4350 3750 4350 4400
-Connection ~ 4350 4400
+	1    0    0    -1
+$EndComp
 $EndSCHEMATC
